File: RFMduino.kicad_pcb (KiCad board)
At the start: 2 copper layers, 68.6 x 53.3 mm, 21 parts, among them J1 Conn_01x02_Male, J2 Conn_01x04_Female, J3 CONN_01, J4 1053354-1, Q1 BSS138, U1 LM1117-3.3, U2 HEX_CONVERTER, U3 RFM69HCW-915

Commit message: corrected pcb
Parts:
- added R5: 10k, Resistor_SMD:R_0603_1608Metric, F.Cu at (136.4, 78.0)
- added R6: 10k, Resistor_SMD:R_0603_1608Metric, F.Cu at (140.6, 78.0)
- Q1, R3, R4: moved to B.Cu
- moved J4 58.7 mm to (183.1, 92.7)
- moved J3 44.8 mm to (176.2, 92.5)
- moved C4 35.9 mm to (169.1, 86.0), turned to 270 degrees
- moved J2 34.6 mm to (139.9, 81.3)
- moved Q1 17.5 mm to (161.7, 75.1)
- moved R4 17.4 mm to (158.7, 75.4), turned to 90 degrees
- moved C3 16.4 mm to (171.2, 72.2)
- moved R1 16.3 mm to (173.7, 86.4)
- moved U2 15.4 mm to (175.4, 78.6)
- moved U3 14.9 mm to (158.7, 85.5), turned to 0 degrees
- moved C1 13.0 mm to (143.3, 66.5)
- moved J1 11.6 mm to (140.0, 69.1), turned to 270 degrees
- moved R2 10.4 mm to (176.6, 86.4)
- moved U1 4.25 mm to (147.4, 71.4)
- moved C2 2.47 mm to (144.9, 76.3), turned to 0 degrees
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Routing:
- net /MISO_3V3: track 39.8 -> 13.5 mm, vias 2 -> 1
- net 5V: track 96.9 -> 121.1 mm, vias 3 -> 2
- net /RST_5V: track 51.1 -> 29.6 mm
- net /MISO_5V: track 7.22 -> 25.2 mm
- net /CS_3V3: track 17.9 -> 35.9 mm, vias 3 -> 2
- net /SCK_5V: track 27.7 -> 11.9 mm, vias 2 -> 1
- net /MOSI_5V: track 36.4 -> 20.9 mm
- net /SCK_3V3: track 10.3 -> 25.5 mm
- net /RST_3V3: track 16.0 -> 31.1 mm
- net +3V3: track 71.3 -> 59.5 mm, vias 4 -> 2
- net /SDA: track 36.9 -> 25.5 mm
- net VCC: track 40.4 -> 51.6 mm, vias 0 -> 2
- net /CS_5V: track 41.5 -> 31.4 mm, vias 2 -> 0
- net Earth: track 202.7 -> 194.3 mm, vias 4 -> 2
- net /SCL: track 37.5 -> 29.3 mm
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