File: RFMduino.sch (KiCad schematic (older format))
At the start: 17 parts, among them J1 Conn_01x02_Male, J2 Conn_01x04_Female, J3 CONN_01, J4 1053354-1, Q1 BSS138, U1 LM1117-3.3, U2 HEX_CONVERTER, U3 RFM69HCW-915

Commit message: corrected pcb
Parts:
- added R5, R6: 10k, Resistor_SMD:R_0603_1608Metric, symbol RFMduino-rescue:10KOHM-0603-1_10W-1%-SparkFun-Resistors
- B1: symbol SparkFun-Boards:ARDUINO_UNO_R3 -> RFMduino-rescue:ARDUINO_UNO_R3-SparkFun-Boards
- C1, C2, C3: symbol SparkFun-Capacitors:0.1UF-0603-25V-_+80_-20%_ -> RFMduino-rescue:0.1UF-0603-25V-_+80_-20%_-SparkFun-Capacitors
- C4: symbol SparkFun-Capacitors:10UF-0603-6.3V-20% -> RFMduino-rescue:10UF-0603-6.3V-20%-SparkFun-Capacitors
- J3: symbol SparkFun-Connectors:CONN_01 -> RFMduino-rescue:CONN_01-SparkFun-Connectors
- J4: symbol 1053354-1:1053354-1 -> RFMduino-rescue:1053354-1-1053354-1
- R1, R2: symbol SparkFun-Resistors:100KOHM-0603-1_10W-1% -> RFMduino-rescue:100KOHM-0603-1_10W-1%-SparkFun-Resistors
- R3, R4: symbol SparkFun-Resistors:10KOHM-0603-1_10W-1% -> RFMduino-rescue:10KOHM-0603-1_10W-1%-SparkFun-Resistors
- U2: symbol SparkFun-IC-Comms:HEX_CONVERTER -> RFMduino-rescue:HEX_CONVERTER-SparkFun-IC-Comms
- U3: symbol SparkFun-RF:RFM69HCW-915 -> RFMduino-rescue:RFM69HCW-915-SparkFun-RF
Connections:
- net 5V: now also R5.1, R6.1
- net SCL: now also R5.2
- net SDA: now also R6.2
Changed lines of the file:
@@
 $EndComp
 $Comp
-L SparkFun-Boards:ARDUINO_UNO_R3 B1
+L RFMduino-rescue:ARDUINO_UNO_R3-SparkFun-Boards B1
 U 1 1 5FF5CDB0
 P 4000 3150
@@
 $EndComp
 $Comp
-L SparkFun-Capacitors:0.1UF-0603-25V-_+80_-20%_ C2
+L RFMduino-rescue:0.1UF-0603-25V-_+80_-20%_-SparkFun-Capacitors C2
 U 1 1 5FF71844
 P 3950 5500
@@
 $EndComp
 $Comp
-L SparkFun-Capacitors:0.1UF-0603-25V-_+80_-20%_ C1
+L RFMduino-rescue:0.1UF-0603-25V-_+80_-20%_-SparkFun-Capacitors C1
 U 1 1 5FF73E0B
 P 3000 5500
@@
 $EndComp
 $Comp
-L SparkFun-Capacitors:0.1UF-0603-25V-_+80_-20%_ C3
+L RFMduino-rescue:0.1UF-0603-25V-_+80_-20%_-SparkFun-Capacitors C3
 U 1 1 5FF800AD
 P 5250 5450
@@
 	6800 5200 6900 5200
 $Comp
-L SparkFun-IC-Comms:HEX_CONVERTER U2
+L RFMduino-rescue:HEX_CONVERTER-SparkFun-IC-Comms U2
 U 1 1 5FF6FA17
 P 6400 5500
@@
 $EndComp
 $Comp
-L SparkFun-Capacitors:10UF-0603-6.3V-20% C4
+L RFMduino-rescue:10UF-0603-6.3V-20%-SparkFun-Capacitors C4
 U 1 1 5FF94EA3
 P 7200 2950
@@
 	9000 3400 8950 3400
 $Comp
-L SparkFun-RF:RFM69HCW-915 U3
+L RFMduino-rescue:RFM69HCW-915-SparkFun-RF U3
 U 1 1 5FF9D9F9
 P 8450 3000
@@
 CS_5V
 $Comp
-L SparkFun-Resistors:100KOHM-0603-1_10W-1% R1
+L RFMduino-rescue:100KOHM-0603-1_10W-1%-SparkFun-Resistors R1
 U 1 1 5FFB09FC
 P 4750 5250
@@
 $EndComp
 $Comp
-L SparkFun-Resistors:100KOHM-0603-1_10W-1% R2
+L RFMduino-rescue:100KOHM-0603-1_10W-1%-SparkFun-Resistors R2
 U 1 1 5FFB5913
 P 4950 5350
@@
 	4400 5550 4950 5550
 $Comp
-L SparkFun-PowerSymbols:5V #SUPPLY01
+L RFMduino-rescue:5V-SparkFun-PowerSymbols #SUPPLY01
 U 1 1 5FFB93A2
 P 3100 3050
@@
 	3500 3050 3100 3050
 $Comp
-L SparkFun-PowerSymbols:5V #SUPPLY02
+L RFMduino-rescue:5V-SparkFun-PowerSymbols #SUPPLY02
 U 1 1 5FFBC18F
 P 4750 5000
@@
 $EndComp
 $Comp
-L SparkFun-PowerSymbols:5V #SUPPLY03
+L RFMduino-rescue:5V-SparkFun-PowerSymbols #SUPPLY03
 U 1 1 5FFBD172
 P 4950 5000
@@
 	8950 3300 9550 3300
 $Comp
-L 1053354-1:1053354-1 J4
+L RFMduino-rescue:1053354-1-1053354-1 J4
 U 1 1 5FFC4663
 P 9750 3300
@@
 Connection ~ 10550 3650
 $Comp
-L SparkFun-Connectors:CONN_01 J3
+L RFMduino-rescue:CONN_01-SparkFun-Connectors J3
 U 1 1 5FFD5DF5
 P 9550 2950
@@
 $EndComp
 $Comp
-L SparkFun-Resistors:10KOHM-0603-1_10W-1% R4
+L RFMduino-rescue:10KOHM-0603-1_10W-1%-SparkFun-Resistors R4
 U 1 1 5FFE7A4F
 P 9400 4600
@@
 $EndComp
 $Comp
-L SparkFun-Resistors:10KOHM-0603-1_10W-1% R3
+L RFMduino-rescue:10KOHM-0603-1_10W-1%-SparkFun-Resistors R3
 U 1 1 5FFECF5C
 P 8500 4600
@@
 	9800 4900 9400 4900
 $Comp
-L SparkFun-PowerSymbols:5V #SUPPLY05
+L RFMduino-rescue:5V-SparkFun-PowerSymbols #SUPPLY05
 U 1 1 5FFFCCB4
 P 8500 4300
@@
 	1    0    0    -1
 $EndComp
-Wire Wire Line
-	5950 1200 5750 1200
-Wire Wire Line
-	5950 1300 5750 1300
 Text Label 5750 1200 0    50   ~ 0
 SDA
@@
 SCL
 $Comp
-L SparkFun-PowerSymbols:5V #SUPPLY04
+L RFMduino-rescue:5V-SparkFun-PowerSymbols #SUPPLY04
 U 1 1 6001E45F
 P 5600 1400
@@
 Wire Wire Line
 	3450 4250 3450 4300
+$Comp
+L RFMduino-rescue:10KOHM-0603-1_10W-1%-SparkFun-Resistors R6
+U 1 1 60353210
+P 5300 1000
+F 0 "R6" V 5258 1068 45  0000 L CNN
+F 1 "10k" V 5342 1068 45  0000 L CNN
+F 2 "Resistor_SMD:R_0603_1608Metric" H 5300 1150 20  0001 C CNN
+F 3 "" H 5300 1000 60  0001 C CNN
+F 4 "RES-00824" V 5384 1068 60  0001 L CNN "Field4"
+	1    5300 1000
+	0    -1   1    0
+$EndComp
+$Comp
+L RFMduino-rescue:10KOHM-0603-1_10W-1%-SparkFun-Resistors R5
+U 1 1 60355089
+P 5000 1100
+F 0 "R5" V 4958 1168 45  0000 L CNN
+F 1 "10k" V 5042 1168 45  0000 L CNN
+F 2 "Resistor_SMD:R_0603_1608Metric" H 5000 1250 20  0001 C CNN
+F 3 "" H 5000 1100 60  0001 C CNN
+F 4 "RES-00824" V 5084 1168 60  0001 L CNN "Field4"
+	1    5000 1100
+	0    -1   1    0
+$EndComp
+Wire Wire Line
+	5300 1200 5950 1200
+Wire Wire Line
+	5000 1300 5950 1300
+$Comp
+L RFMduino-rescue:5V-SparkFun-PowerSymbols #SUPPLY0101
+U 1 1 6035AD8B
+P 5300 700
+F 0 "#SUPPLY0101" H 5350 700 45  0001 L BNN
+F 1 "5V" H 5300 870 45  0000 C CNN
+F 2 "XXX-00000" H 5300 881 60  0001 C CNN
+F 3 "" H 5300 700 60  0001 C CNN
+	1    5300 700
+	1    0    0    -1
+$EndComp
+Wire Wire Line
+	5300 800  5300 700
+$Comp
+L RFMduino-rescue:5V-SparkFun-PowerSymbols #SUPPLY0102
+U 1 1 60360DE2
+P 5000 700
+F 0 "#SUPPLY0102" H 5050 700 45  0001 L BNN
+F 1 "5V" H 5000 870 45  0000 C CNN
+F 2 "XXX-00000" H 5000 881 60  0001 C CNN
+F 3 "" H 5000 700 60  0001 C CNN
+	1    5000 700
+	1    0    0    -1
+$EndComp
+Wire Wire Line
+	5000 700  5000 900
 $EndSCHEMATC
